File: Breadboard Power Supply.kicad_pcb (KiCad board)
At the start: 2 copper layers, 30.1 x 52.1 mm, 15 parts, among them J1 Barrel_Jack_Switch, J2 Conn_02x02_Odd_Even, J3 Conn_02x02_Odd_Even, SW1 SW_DPDT_x2, U1 LM7805_TO220

Commit message: 102. video yarıda kaldı
Parts:
- moved J1 78.8 mm to (90.6, 150.9), turned to 270 degrees
- moved R2 70.9 mm to (151.0, 134.2)
- moved J3 66.2 mm to (101.5, 152.7)
- moved C1 57.1 mm to (121.9, 138.6)
- moved D1 57.1 mm to (106.3, 137.9)
- moved D3 57.1 mm to (106.3, 142.2)
- moved D5 57.1 mm to (132.6, 136.6)
- moved U1 57.1 mm to (134.1, 122.7)
- moved C2 57.1 mm to (145.2, 122.7)
- moved D2 57.1 mm to (118.8, 120.9)
- moved D4 57.1 mm to (118.8, 125.1)
- moved SW1 49.5 mm to (95.2, 131.2), turned to 90 degrees
- moved D6 41.2 mm to (94.1, 118.1)
- moved R1 40.0 mm to (109.3, 117.9), turned to 180 degrees
- moved J2 21.1 mm to (101.5, 107.7)

Commit message: 102 bitti
Parts:
- moved R2 64.2 mm to (89.4, 116.1), turned to 270 degrees
- moved C2 56.8 mm to (90.0, 109.2)
- moved U1 54.5 mm to (79.6, 121.7)
- moved C1 50.4 mm to (79.6, 111.1)
- moved D4 41.2 mm to (78.2, 131.9)
- moved D2 41.1 mm to (78.2, 127.1)
- moved R1 40.0 mm to (96.1, 155.6), turned to 90 degrees
- moved D5 38.4 mm to (94.5, 141.4)
- moved D1 28.1 mm to (78.2, 136.7)
- moved D3 28.1 mm to (78.2, 141.5)
- moved SW1 2.07 mm to (95.1, 133.3)
- moved D6 1.82 mm to (94.5, 119.9)

Commit message: 103. video ortada kaldı
Routing:
- net /BJ_pin2: track 0.00 -> 11.0 mm

Commit message: 104. video tamamlandı
Parts:
- moved R1 32.8 mm to (89.5, 123.4)
- moved R2 32.0 mm to (94.9, 147.6)
Routing:
- net /GND: track 0.00 -> 88.6 mm
- net /Vout2: track 0.00 -> 69.2 mm
- net /Vout1: track 0.00 -> 48.7 mm
- net /Vin: track 0.00 -> 31.5 mm
- net /BJ_pin1: track 0.00 -> 29.2 mm
- net Net-(D5-Pad2): track 0.00 -> 14.7 mm
- net /BJ_pin2: track 11.0 -> 25.1 mm
- net Net-(D6-Pad2): track 0.00 -> 10.1 mm
- added copper zone on B.Cu, net /GND
Changed lines of the file:
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@@
-(kicad_pcb (version 20171130) (host pcbnew "(5.1.10)-1")
+(kicad_pcb (version 20171130) (host pcbnew 5.1.10)
   (general
     (thickness 1.6)
     (drawings 8)
-    (tracks 2)
+    (tracks 68)
     (zones 0)
     (modules 15)
@@
     (pad_to_mask_clearance 0)
     (aux_axis_origin 0 0)
-    (visible_elements 7FFFFFFF)
+    (visible_elements 7FFFF7FF)
     (pcbplotparams
       (layerselection 0x010fc_ffffffff)
@@
   )
   (module Resistor_THT:R_Axial_DIN0207_L6.3mm_D2.5mm_P7.62mm_Horizontal (layer F.Cu)
-    (at 96.139 155.575 90)
+    (at 89.535 123.444 90)
     (descr "Resistor, Axial_DIN0207 series, Axial, Horizontal, pin pitch=7.62mm, 0.25W = 1/4W, length*diameter=6.3*2.5mm^2, http://cdn-reichelt.de/documents/datenblatt/B400/1_4W%23YAG.pdf")
     (tags "Resistor Axial_DIN0207 series Axial Horizontal pin pitch 7.62mm 0.25W = 1/4W length 6.3mm diameter 2.5mm")
@@
       (effects (font (size 1 1) (thickness 0.15)))
     )
-    (fp_text value "560 Ω" (at 4.318 -2.667 270) (layer F.Fab)
+    (fp_text value "560 Ω" (at 4.191 -2.286 270) (layer F.Fab)
       (effects (font (size 1 1) (thickness 0.15)))
     )
@@
   )
   (module Resistor_THT:R_Axial_DIN0207_L6.3mm_D2.5mm_P7.62mm_Horizontal (layer F.Cu)
-    (at 89.408 116.078 270)
+    (at 94.869 147.574 270)
     (descr "Resistor, Axial_DIN0207 series, Axial, Horizontal, pin pitch=7.62mm, 0.25W = 1/4W, length*diameter=6.3*2.5mm^2, http://cdn-reichelt.de/documents/datenblatt/B400/1_4W%23YAG.pdf")
     (tags "Resistor Axial_DIN0207 series Axial Horizontal pin pitch 7.62mm 0.25W = 1/4W length 6.3mm diameter 2.5mm")
@@
       (effects (font (size 1 1) (thickness 0.15)))
     )
-    (fp_text value "560 Ω" (at 9.652 0 180) (layer F.Fab)
+    (fp_text value "560 Ω" (at 3.81 2.413 270) (layer F.Fab)
       (effects (font (size 1 1) (thickness 0.15)))
     )
@@
   (gr_line (start 76.2 157.48) (end 106.299 157.48) (layer Edge.Cuts) (width 0.05))
   (gr_line (start 76.2 105.41) (end 76.2 157.48) (layer Edge.Cuts) (width 0.05))
+  (segment (start 78.232 141.478) (end 78.232 136.685667) (width 0.3) (layer F.Cu) (net 1))
+  (segment (start 78.232 136.685667) (end 78.232 135.636) (width 0.3) (layer F.Cu) (net 1))
+  (segment (start 78.232 135.636) (end 80.264 133.604) (width 0.3) (layer F.Cu) (net 1))
+  (segment (start 80.264 122.301) (end 79.629 121.666) (width 0.3) (layer F.Cu) (net 1))
+  (segment (start 80.264 133.604) (end 80.264 122.301) (width 0.3) (layer F.Cu) (net 1))
+  (segment (start 79.629 121.666) (end 79.629 111.07) (width 0.3) (layer F.Cu) (net 1))
+  (segment (start 104.013 155.194) (end 101.473 155.194) (width 0.3) (layer B.Cu) (net 2))
+  (segment (start 101.473 155.194) (end 98.425 152.146) (width 0.3) (layer B.Cu) (net 2))
+  (segment (start 98.425 145.288) (end 94.488 141.351) (width 0.3) (layer B.Cu) (net 2))
+  (segment (start 98.425 152.146) (end 98.425 145.288) (width 0.3) (layer B.Cu) (net 2))
+  (segment (start 94.488 140.151) (end 91.313 136.976) (width 0.3) (layer B.Cu) (net 2))
+  (segment (start 94.488 141.351) (end 94.488 140.151) (width 0.3) (layer B.Cu) (net 2))
+  (segment (start 91.313 134.814334) (end 88.392 131.893334) (width 0.3) (layer B.Cu) (net 2))
+  (segment (start 91.313 136.976) (end 91.313 134.814334) (width 0.3) (layer B.Cu) (net 2))
+  (segment (start 88.392 131.893334) (end 88.392 127.101001) (width 0.3) (layer B.Cu) (net 2))
+  (segment (start 94.488 121.005001) (end 94.488 119.888) (width 0.3) (layer B.Cu) (net 2))
+  (segment (start 88.392 127.101001) (end 94.488 121.005001) (width 0.3) (layer B.Cu) (net 2))
+  (segment (start 87.604001 127.101001) (end 82.169 121.666) (width 0.3) (layer B.Cu) (net 2))
+  (segment (start 88.392 127.101001) (end 87.604001 127.101001) (width 0.3) (layer B.Cu) (net 2))
+  (segment (start 92.543 109.22) (end 92.543 108.037) (width 0.3) (layer B.Cu) (net 2))
+  (segment (start 92.543 108.037) (end 91.948 107.442) (width 0.3) (layer B.Cu) (net 2))
+  (segment (start 88.257 107.442) (end 84.629 111.07) (width 0.3) (layer B.Cu) (net 2))
+  (segment (start 91.948 107.442) (end 88.257 107.442) (width 0.3) (layer B.Cu) (net 2))
+  (segment (start 84.629 111.07) (end 82.423 113.276) (width 0.3) (layer B.Cu) (net 2))
+  (segment (start 82.423 121.412) (end 82.169 121.666) (width 0.3) (layer B.Cu) (net 2))
+  (segment (start 82.423 113.276) (end 82.423 121.412) (width 0.3) (layer B.Cu) (net 2))
+  (segment (start 101.473 110.236) (end 104.013 110.236) (width 0.3) (layer B.Cu) (net 2))
+  (segment (start 93.559 110.236) (end 92.543 109.22) (width 0.3) (layer B.Cu) (net 2))
+  (segment (start 101.473 110.236) (end 93.559 110.236) (width 0.3) (layer B.Cu) (net 2))
+  (segment (start 84.709 120.777) (end 84.709 121.666) (width 0.3) (layer B.Cu) (net 3))
+  (segment (start 84.709 121.666) (end 84.709 117.729) (width 0.3) (layer B.Cu) (net 3))
+  (segment (start 90.043 112.395) (end 90.043 109.22) (width 0.3) (layer B.Cu) (net 3))
+  (segment (start 84.709 117.729) (end 90.043 112.395) (width 0.3) (layer B.Cu) (net 3))
+  (segment (start 94.869 147.574) (end 92.583 145.288) (width 0.3) (layer F.Cu) (net 3))
+  (segment (start 94.912998 130.7535) (end 95.123 130.7535) (width 0.3) (layer F.Cu) (net 3))
+  (segment (start 92.583 133.083498) (end 94.912998 130.7535) (width 0.3) (layer F.Cu) (net 3))
+  (segment (start 92.583 145.288) (end 92.583 133.083498) (width 0.3) (layer F.Cu) (net 3))
+  (segment (start 84.709 121.666) (end 85.471 121.666) (width 0.3) (layer F.Cu) (net 3))
+  (segment (start 93.4015 129.032) (end 95.123 130.7535) (width 0.3) (layer F.Cu) (net 3))
+  (segment (start 92.837 129.032) (end 93.4015 129.032) (width 0.3) (layer F.Cu) (net 3))
+  (segment (start 85.471 121.666) (end 92.837 129.032) (width 0.3) (layer F.Cu) (net 3))
+  (segment (start 90.551 138.844667) (end 88.392 136.685667) (width 0.3) (layer F.Cu) (net 4))
+  (segment (start 90.551 150.876) (end 90.551 138.844667) (width 0.3) (layer F.Cu) (net 4))
+  (segment (start 78.807334 127.101001) (end 88.392 136.685667) (width 0.3) (layer B.Cu) (net 4))
+  (segment (start 78.232 127.101001) (end 78.807334 127.101001) (width 0.3) (layer B.Cu) (net 4))
   (segment (start 84.551 145.319) (end 88.392 141.478) (width 0.3) (layer B.Cu) (net 5))
   (segment (start 84.551 150.876) (end 84.551 145.319) (width 0.3) (layer B.Cu) (net 5))
+  (segment (start 78.807334 131.893334) (end 78.232 131.893334) (width 0.3) (layer B.Cu) (net 5))
+  (segment (start 88.392 141.478) (end 78.807334 131.893334) (width 0.3) (layer B.Cu) (net 5))
+  (segment (start 97.028 153.035) (end 94.869 155.194) (width 0.3) (layer F.Cu) (net 6))
+  (segment (start 97.028 141.351) (end 97.028 153.035) (width 0.3) (layer F.Cu) (net 6))
+  (segment (start 90.043 115.443) (end 89.408 116.078) (width 0.3) (layer B.Cu) (net 7))
+  (segment (start 92.964 115.824) (end 97.028 119.888) (width 0.3) (layer B.Cu) (net 7))
+  (segment (start 89.535 115.824) (end 92.964 115.824) (width 0.3) (layer B.Cu) (net 7))
+  (segment (start 101.473 152.654) (end 104.013 152.654) (width 0.3) (layer F.Cu) (net 9))
+  (segment (start 104.013 107.696) (end 101.473 107.696) (width 0.3) (layer F.Cu) (net 9))
+  (segment (start 101.473 107.696) (end 99.06 107.696) (width 0.3) (layer F.Cu) (net 9))
+  (segment (start 95.123 133.2535) (end 94.9655 133.2535) (width 0.3) (layer F.Cu) (net 9))
+  (segment (start 95.123 133.2535) (end 98.679 136.8095) (width 0.3) (layer F.Cu) (net 9))
+  (segment (start 100.801235 152.654) (end 101.473 152.654) (width 0.3) (layer F.Cu) (net 9))
+  (segment (start 98.679 150.531765) (end 100.801235 152.654) (width 0.3) (layer F.Cu) (net 9))
+  (segment (start 89.535 123.444) (end 97.79 123.444) (width 0.3) (layer F.Cu) (net 9))
+  (segment (start 98.679 124.333) (end 98.679 137.16) (width 0.3) (layer F.Cu) (net 9))
+  (segment (start 97.79 123.444) (end 98.679 124.333) (width 0.3) (layer F.Cu) (net 9))
+  (segment (start 98.679 137.16) (end 98.679 150.531765) (width 0.3) (layer F.Cu) (net 9))
+  (segment (start 98.679 136.8095) (end 98.679 137.16) (width 0.3) (layer F.Cu) (net 9))
+  (segment (start 99.06 107.696) (end 98.679 108.077) (width 0.3) (layer F.Cu) (net 9))
+  (segment (start 98.679 108.077) (end 98.679 124.333) (width 0.3) (layer F.Cu) (net 9))
+  (zone (net 2) (net_name /GND) (layer B.Cu) (hatch edge 0.508)
+    (connect_pads (clearance 0.508))
+    (min_thickness 0.254)
+    (fill yes (arc_segments 32) (thermal_gap 0.508) (thermal_bridge_width 0.508))
+    (polygon
+      (pts
+        (xy 106.172 112.395) (xy 99.06 112.395) (xy 99.06 150.495) (xy 106.172 150.495) (xy 106.045 157.353)
+        (xy 76.327 157.353) (xy 76.327 105.537) (xy 106.172 105.537)
+      )
+    )
+  )
 )
